Commit message: Finished: modify the urdf and xacro file for moving target and mobile sensors, so we have a nice-looking demonstration.

File: models/motion_lamp.urdf.xacro (robot description, xacro)
@@ -1,6 +1,5 @@
 <?xml version="1.0" ?>
 <robot name="turtlebot3_burger" xmlns:xacro="http://ros.org/wiki/xacro">
-  <xacro:include filename="$(find turtlebot3_description)/urdf/common_properties.xacro"/>
-  <xacro:include filename="$(find turtlebot3_description)/urdf/turtlebot3_burger.gazebo.xacro"/>
+  <xacro:include filename="$(find fim_track)/models/motion_lamp.gazebo.xacro"/>
   <link name="base_footprint"/>
   <joint name="base_joint" type="fixed">
@@ -15,5 +14,4 @@
         <mesh filename="package://turtlebot3_description/meshes/bases/burger_base.stl" scale="0.001 0.001 0.001"/>
       </geometry>
-      <material name="light_black"/>
     </visual>
     <collision>
@@ -43,5 +41,4 @@
         <mesh filename="package://turtlebot3_description/meshes/wheels/left_tire.stl" scale="0.001 0.001 0.001"/>
       </geometry>
-      <material name="dark"/>
     </visual>
     <collision>
@@ -71,5 +68,4 @@
         <mesh filename="package://turtlebot3_description/meshes/wheels/right_tire.stl" scale="0.001 0.001 0.001"/>
       </geometry>
-      <material name="dark"/>
     </visual>
     <collision>
@@ -122,7 +118,6 @@
       <origin xyz="0 0 0.0" rpy="0 0 0"/>
       <geometry>
-	<mesh filename="model://lamp_post/meshes/lamp_post.dae" scale="0.4 0.4 0.4"/>
-	</geometry>
-      <material name="RedBright"/>
+    	<mesh filename="package://turtlebot3_description/meshes/sensors/lds.stl" scale="0.001 0.001 0.001"/>
+  	</geometry>
     </visual>
     <collision>

File: models/turtlebot3_burger.urdf.xacro (robot description, xacro)
@@ -2,5 +2,5 @@
 <robot name="turtlebot3_burger" xmlns:xacro="http://ros.org/wiki/xacro">
   <xacro:include filename="$(find turtlebot3_description)/urdf/common_properties.xacro"/>
-  <xacro:include filename="$(find turtlebot3_description)/urdf/turtlebot3_burger.gazebo.xacro"/>
+<xacro:include filename="$(find fim_track)/models/turtlebot3_burger.gazebo.xacro"/>
   <link name="base_footprint"/>
   <joint name="base_joint" type="fixed">
